File: ebus-adapter/ebus-adapter.sch (KiCad schematic (older format))
At the start: 25 parts, among them J1 EBus-Connector, J2 Serial, Q1 BC337, U1 L7805, U2 LM393N, U3 4N25, U4 4N25

Commit message: Corrected footprint of 7805 voltage ragulator
Parts:
- U1: value L7805 -> L78L05; footprint Package_TO_SOT_THT:TO-92L_Inline -> Package_TO_SOT_THT:TO-92_Inline; symbol Regulator_Linear:L7805 -> Regulator_Linear:MC78L05_TO92
Connections:
- net +5V: now also U1.1 (VO); no longer U1.3 (OUT)
- net at C1.1, D1.1 (K), D2.1 (K)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: now also U1.3 (VI); no longer U1.1 (IN)
Changed lines of the file:
@@
 $EndComp
 $Comp
-L Regulator_Linear:L7805 U1
+L Regulator_Linear:MC78L05_TO92 U1
 U 1 1 5FCE71F1
 P 3150 2050
 F 0 "U1" H 3150 2292 50  0000 C CNN
-F 1 "L7805" H 3150 2201 50  0000 C CNN
-F 2 "Package_TO_SOT_THT:TO-92L_Inline" H 3175 1900 50  0001 L CIN
+F 1 "L78L05" H 3150 2201 50  0000 C CNN
+F 2 "Package_TO_SOT_THT:TO-92_Inline" H 3175 1900 50  0001 L CIN
 F 3 "http://www.st.com/content/ccc/resource/technical/document/datasheet/41/4f/b3/b0/12/d4/47/88/CD00000444.pdf/files/CD00000444.pdf/jcr:content/translations/en.CD00000444.pdf" H 3150 2000 50  0001 C CNN
 	1    3150 2050
